Commit message: Added wrenchs to box model

File: ur_gazebo/models/box.urdf (robot description, URDF)
Before this commit: robot MBZIRC_box, 3 links, 2 joints
Links:
- added link wrench_1, mass 0.01; collision cylinder length=0.12 radius=0.01; visual mesh filename=package://ur_gazebo/models/llave12.dae
- added link wrench_2, mass 0.01; collision cylinder length=0.19 radius=0.01; visual mesh filename=package://ur_gazebo/models/llave19.stl
- added link wrench_3, mass 0.01; collision cylinder length=0.16 radius=0.01; visual mesh filename=package://ur_gazebo/models/llave16.stl
- link box_handle: geometry collision box size=0.0185 0.06 0.0185; visual box size=0.0185 0.06 0.0185
Joints:
- added joint fixed_joint_3: type fixed, parent box, child wrench_1, origin xyz=0.4 -0.42 0.3 rpy=0.0 0.0 0.0 
- added joint fixed_joint_4: type fixed, parent box, child wrench_2, origin xyz=0.3 -0.42 0.32 rpy=0.0 0.0 0.0 
- added joint fixed_joint_5: type fixed, parent box, child wrench_3, origin xyz=0.25 -0.42 0.31 rpy=0.0 0.0 0.0 
