Commit message: Added hokuyo in tcp

File: ur_description/urdf/ur5.urdf.xacro (robot description, xacro)
@@ -251,5 +251,5 @@
       </xacro:unless>
       <xacro:if value="${joint_limited}">
-        <limit lower="${-pi}" upper="${pi}" effort="28.0" velocity="3.2"/>
+        <limit lower="${-2.0 * pi}" upper="${2.0 * pi}" effort="28.0" velocity="3.2"/>
       </xacro:if>
       <dynamics damping="0.0" friction="0.0"/>
@@ -306,4 +306,95 @@
       <child link="${prefix}tool0"/>
     </joint>
+   <joint name="gripper_joint" type="fixed">
+    <axis xyz="0 1 0" />
+    <origin xyz="0.105 0.0 0.0" rpy="0 0 0"/>
+    <parent link="${prefix}ee_link"/>
+    <child link="gripper"/>
+  </joint>
+  <link name="gripper">
+    <visual>
+      <origin xyz="0 0 0" rpy="0 0 0" />
+      <geometry>
+          <box size="0.21 0.065 0.04"/>
+      </geometry>
+     <material name="black">
+        <color rgba="0.05 0.05 0.05 1"/>
+      </material>
+    </visual>
+	<collision>
+		<origin xyz="0 0 0" rpy="0 0 0" />
+		<geometry>
+          <box size="0.21 0.065 0.04"/>
+		</geometry>
+	</collision>
+	<inertial>
+		<mass value="0.01" />
+		<inertia ixx="0.01" ixy="0.0" ixz="0.0"
+				iyy="0.01" iyz="0.0"
+				izz="0.01" />
+	</inertial>
+  </link>
+  <joint name="hokuyo_joint" type="fixed">
+    <axis xyz="0 1 0" />
+    <origin xyz="-0.05 0.0 0.03" rpy="0 0 0"/>
+    <parent link="gripper"/>
+    <child link="hokuyo_link"/>
+  </joint>
+  <!-- Hokuyo Laser -->
+  <link name="hokuyo_link">
+    <collision>
+      <origin xyz="0 0 0" rpy="0 0 0"/>
+      <geometry>
+    <box size="0.1 0.1 0.1"/>
+      </geometry>
+    </collision>
+    <visual>
+      <origin xyz="0 0 0" rpy="0 0 0"/>
+      <geometry>
+        <mesh filename="package://ur_description/meshes/hokuyo.dae"/>
+      </geometry>
+    </visual>
+    <inertial>
+      <mass value="1e-5" />
+      <origin xyz="0 0 0" rpy="0 0 0"/>
+      <inertia ixx="1e-6" ixy="0" ixz="0" iyy="1e-6" iyz="0" izz="1e-6" />
+    </inertial>
+  </link>
+  <!-- hokuyo -->
+  <gazebo reference="hokuyo_link">
+    <sensor type="gpu_ray" name="head_hokuyo_sensor">
+      <pose>0 0 0 0 0 0</pose>
+      <visualize>false</visualize>
+      <update_rate>40</update_rate>
+      <ray>
+        <scan>
+          <horizontal>
+            <samples>720</samples>
+            <resolution>1</resolution>
+            <min_angle>-1.570796</min_angle>
+            <max_angle>1.570796</max_angle>
+          </horizontal>
+        </scan>
+        <range>
+          <min>0.10</min>
+          <max>2.0</max>
+          <resolution>0.01</resolution>
+        </range>
+        <noise>
+          <type>gaussian</type>
+          <!-- Noise parameters based on published spec for Hokuyo laser
+               achieving "+-30mm" accuracy at range < 10m.  A mean of 0.0m and
+               stddev of 0.01m will put 99.7% of samples within 0.03m of the true
+               reading. -->
+          <mean>0.0</mean>
+          <stddev>0.01</stddev>
+        </noise>
+      </ray>
+      <plugin name="gazebo_ros_head_hokuyo_controller" filename="libgazebo_ros_gpu_laser.so">
+        <topicName>/hokuyo/laser/scan</topicName>
+        <frameName>hokuyo_link</frameName>
+      </plugin>
+    </sensor>
+  </gazebo>
   </xacro:macro>
 </robot>

Commit message: Added mobile_base

File: ur_description/urdf/ur5.urdf.xacro (robot description, xacro)
@@ -69,4 +69,33 @@
   </xacro:macro>
   <xacro:macro name="ur5_robot" params="prefix joint_limited">
+   <link name="${prefix}mobile_base">
+    <visual>
+      <origin xyz="0 0 0" rpy="0 0 0" />
+      <geometry>
+          <box size="0.6 0.4 0.3"/>
+      </geometry>
+     <material name="black">
+        <color rgba="0.05 0.05 0.05 1"/>
+      </material>
+    </visual>
+	<collision>
+		<origin xyz="0 0 0" rpy="0 0 0" />
+		<geometry>
+          <box size="0.6 0.4 0.3"/>
+		</geometry>
+	</collision>
+	<inertial>
+		<mass value="100" />
+		<inertia ixx="1" ixy="0.0" ixz="0.0"
+				iyy="1" iyz="0.0"
+				izz="1" />
+	</inertial>
+  </link>
+  <joint name="${prefix}base_joint" type="fixed">
+    <axis xyz="0 0 1" />
+    <origin xyz="0.0 0.0 0.15" rpy="0 0 0"/>
+    <parent link="${prefix}mobile_base"/>
+    <child link="${prefix}base_link"/>
+  </joint>
     <link name="${prefix}base_link" >
       <visual>
@@ -251,5 +280,5 @@
       </xacro:unless>
       <xacro:if value="${joint_limited}">
-        <limit lower="${-2.0 * pi}" upper="${2.0 * pi}" effort="28.0" velocity="3.2"/>
+        <limit lower="${-1.9 * pi}" upper="${1.9 * pi}" effort="28.0" velocity="3.2"/>
       </xacro:if>
       <dynamics damping="0.0" friction="0.0"/>
@@ -306,11 +335,11 @@
       <child link="${prefix}tool0"/>
     </joint>
-   <joint name="gripper_joint" type="fixed">
+   <joint name="${prefix}gripper_joint" type="fixed">
     <axis xyz="0 1 0" />
     <origin xyz="0.105 0.0 0.0" rpy="0 0 0"/>
     <parent link="${prefix}ee_link"/>
-    <child link="gripper"/>
+    <child link="${prefix}gripper"/>
   </joint>
-  <link name="gripper">
+  <link name="${prefix}gripper">
     <visual>
       <origin xyz="0 0 0" rpy="0 0 0" />
@@ -335,12 +364,12 @@
 	</inertial>
   </link>
-  <joint name="hokuyo_joint" type="fixed">
+  <joint name="${prefix}hokuyo_joint" type="fixed">
     <axis xyz="0 1 0" />
     <origin xyz="-0.05 0.0 0.03" rpy="0 0 0"/>
-    <parent link="gripper"/>
-    <child link="hokuyo_link"/>
+    <parent link="${prefix}gripper"/>
+    <child link="${prefix}hokuyo_link"/>
   </joint>
   <!-- Hokuyo Laser -->
-  <link name="hokuyo_link">
+  <link name="${prefix}hokuyo_link">
     <collision>
       <origin xyz="0 0 0" rpy="0 0 0"/>
@@ -362,5 +391,5 @@
   </link>
   <!-- hokuyo -->
-  <gazebo reference="hokuyo_link">
+  <gazebo reference="${prefix}hokuyo_link">
     <sensor type="gpu_ray" name="head_hokuyo_sensor">
       <pose>0 0 0 0 0 0</pose>

File: ur_description/urdf/ur5_joint_limited_robot.urdf.xacro (robot description, xacro)
@@ -11,5 +11,5 @@
   <joint name="world_joint" type="fixed">
     <parent link="world" />
-    <child link = "base_link" />
+    <child link = "mobile_base" />
     <origin xyz="0.0 0.0 0.0" rpy="0.0 0.0 0.0" />
   </joint>

File: ur_description/urdf/ur5_robot.urdf.xacro (robot description, xacro)
@@ -11,5 +11,5 @@
   <joint name="world_joint" type="fixed">
     <parent link="world" />
-    <child link = "base_link" />
+    <child link = "mobile_base" />
     <origin xyz="0.0 0.0 0.0" rpy="0.0 0.0 0.0" />
   </joint>

Commit message: Modified files to use mobile base and correct box size

File: ur_description/urdf/ur5.urdf.xacro (robot description, xacro)
@@ -73,5 +73,5 @@
       <origin xyz="0 0 0" rpy="0 0 0" />
       <geometry>
-          <box size="0.6 0.4 0.3"/>
+          <box size="0.83 0.83 0.4"/>
       </geometry>
      <material name="black">
@@ -82,5 +82,5 @@
 		<origin xyz="0 0 0" rpy="0 0 0" />
 		<geometry>
-          <box size="0.6 0.4 0.3"/>
+          <box size="0.83 0.83 0.4"/>
 		</geometry>
 	</collision>
@@ -94,5 +94,5 @@
   <joint name="${prefix}base_joint" type="fixed">
     <axis xyz="0 0 1" />
-    <origin xyz="0.0 0.0 0.15" rpy="0 0 0"/>
+    <origin xyz="0.0 0.0 0.2" rpy="0 0 0"/>
     <parent link="${prefix}mobile_base"/>
     <child link="${prefix}base_link"/>

File: ur_description/urdf/ur5_joint_limited_robot.urdf.xacro (robot description, xacro)
@@ -12,5 +12,5 @@
     <parent link="world" />
     <child link = "mobile_base" />
-    <origin xyz="0.0 0.0 0.0" rpy="0.0 0.0 0.0" />
+    <origin xyz="0.0 0.0 0.2" rpy="0.0 0.0 0.0" />
   </joint>
 </robot>

File: ur_description/urdf/ur5_robot.urdf.xacro (robot description, xacro)
@@ -12,5 +12,5 @@
     <parent link="world" />
     <child link = "mobile_base" />
-    <origin xyz="0.0 0.0 0.0" rpy="0.0 0.0 0.0" />
+    <origin xyz="0.0 0.0 0.2" rpy="0.0 0.0 0.0" />
   </joint>
 </robot>

File: ur_gazebo/models/box.urdf (robot description, URDF)
Before this commit: robot MBZIRC_box, 6 links, 5 joints
Links:
- link box: mass 1.0 -> 100.0; geometry collision box size=1 1 0.75; visual box size=1 1 0.75
- link cyl_handle: geometry collision cylinder length=0.02 radius=0.04; visual cylinder length=0.02 radius=0.04
Joints:
- joint fixed_joint_1: origin xyz=-0.155 -0.42 0.0 rpy=0.0 0.0 0.0  -> xyz=-0.155 -0.51 0.0 rpy=0.0 0.0 0.0 
- joint fixed_joint_3: origin xyz=0.4 -0.42 0.3 rpy=0.0 0.0 0.0  -> xyz=0.4 -0.51 0.225 rpy=0.0 0.0 0.0 
- joint fixed_joint_4: origin xyz=0.3 -0.42 0.32 rpy=0.0 0.0 0.0  -> xyz=0.3 -0.51 0.245 rpy=0.0 0.0 0.0 
- joint fixed_joint_5: origin xyz=0.25 -0.42 0.31 rpy=0.0 0.0 0.0  -> xyz=0.25 -0.51 0.235 rpy=0.0 0.0 0.0 

Commit message: Added mobile base

File: ur_description/urdf/ur5.urdf.xacro (robot description, xacro)
@@ -73,5 +73,5 @@
       <origin xyz="0 0 0" rpy="0 0 0" />
       <geometry>
-          <box size="0.83 0.83 0.4"/>
+          <box size="0.405 0.605 0.345"/>
       </geometry>
      <material name="black">
@@ -82,5 +82,92 @@
 		<origin xyz="0 0 0" rpy="0 0 0" />
 		<geometry>
-          <box size="0.83 0.83 0.4"/>
+          <box size="0.405 0.605 0.345"/>
+		</geometry>
+	</collision>
+	<inertial>
+		<mass value="100" />
+		<inertia ixx="1" ixy="0.0" ixz="0.0"
+				iyy="1" iyz="0.0"
+				izz="1" />
+	</inertial>
+  </link>
+  <joint name="${prefix}right_wheels_joint" type="fixed">
+    <axis xyz="0 0 1" />
+    <origin xyz="0.3025 0.0 0.0275" rpy="0 0 0"/>
+    <parent link="${prefix}mobile_base"/>
+    <child link="${prefix}right_wheels"/>
+  </joint>
+   <link name="${prefix}right_wheels">
+    <visual>
+      <origin xyz="0 0 0" rpy="0 0 0" />
+      <geometry>
+          <box size="0.18 0.605 0.4"/>
+      </geometry>
+     <material name="black">
+        <color rgba="0.05 0.05 0.05 1"/>
+      </material>
+    </visual>
+	<collision>
+		<origin xyz="0 0 0" rpy="0 0 0" />
+		<geometry>
+          <box size="0.18 0.605 0.4"/>
+		</geometry>
+	</collision>
+	<inertial>
+		<mass value="100" />
+		<inertia ixx="1" ixy="0.0" ixz="0.0"
+				iyy="1" iyz="0.0"
+				izz="1" />
+	</inertial>
+  </link>
+  <joint name="${prefix}left_wheels_joint" type="fixed">
+    <axis xyz="0 0 1" />
+    <origin xyz="-0.3025 0.0 0.0275" rpy="0 0 0"/>
+    <parent link="${prefix}mobile_base"/>
+    <child link="${prefix}left_wheels"/>
+  </joint>
+   <link name="${prefix}left_wheels">
+    <visual>
+      <origin xyz="0 0 0" rpy="0 0 0" />
+      <geometry>
+          <box size="0.18 0.605 0.4"/>
+      </geometry>
+     <material name="black">
+        <color rgba="0.05 0.05 0.05 1"/>
+      </material>
+    </visual>
+	<collision>
+		<origin xyz="0 0 0" rpy="0 0 0" />
+		<geometry>
+          <box size="0.18 0.605 0.4"/>
+		</geometry>
+	</collision>
+	<inertial>
+		<mass value="100" />
+		<inertia ixx="1" ixy="0.0" ixz="0.0"
+				iyy="1" iyz="0.0"
+				izz="1" />
+	</inertial>
+  </link>
+  <joint name="${prefix}lidar_joint" type="fixed">
+    <axis xyz="0 0 1" />
+    <origin xyz="0.0 0.3675 0.0" rpy="0 0 0"/>
+    <parent link="${prefix}mobile_base"/>
+    <child link="${prefix}lidar"/>
+  </joint>
+   <link name="${prefix}lidar">
+    <visual>
+      <origin xyz="0 0 0" rpy="0 0 0" />
+      <geometry>
+          <box size="0.405 0.13 0.345"/>
+      </geometry>
+     <material name="black">
+        <color rgba="0.05 0.05 0.05 1"/>
+      </material>
+    </visual>
+	<collision>
+		<origin xyz="0 0 0" rpy="0 0 0" />
+		<geometry>
+          <box size="0.405 0.13 0.345"/>
 		</geometry>
 	</collision>
@@ -94,5 +181,5 @@
   <joint name="${prefix}base_joint" type="fixed">
     <axis xyz="0 0 1" />
-    <origin xyz="0.0 0.0 0.2" rpy="0 0 0"/>
+    <origin xyz="0.0 0.0 0.1725" rpy="0 0 -1.5708"/>
     <parent link="${prefix}mobile_base"/>
     <child link="${prefix}base_link"/>
@@ -345,5 +432,5 @@
       <origin xyz="0 0 0" rpy="0 0 0" />
       <geometry>
-          <box size="0.21 0.065 0.04"/>
+          <box size="0.19 0.065 0.04"/>
       </geometry>
      <material name="black">
@@ -354,5 +441,5 @@
 		<origin xyz="0 0 0" rpy="0 0 0" />
 		<geometry>
-          <box size="0.21 0.065 0.04"/>
+          <box size="0.19 0.065 0.04"/>
 		</geometry>
 	</collision>

File: ur_description/urdf/ur5_joint_limited_robot.urdf.xacro (robot description, xacro)
@@ -12,5 +12,5 @@
     <parent link="world" />
     <child link = "mobile_base" />
-    <origin xyz="0.0 0.0 0.2" rpy="0.0 0.0 0.0" />
+    <origin xyz="0.0 0.0 0.1725" rpy="0.0 0.0 0.0" />
   </joint>
 </robot>

File: ur_description/urdf/ur5_robot.urdf.xacro (robot description, xacro)
@@ -12,5 +12,5 @@
     <parent link="world" />
     <child link = "mobile_base" />
-    <origin xyz="0.0 0.0 0.2" rpy="0.0 0.0 0.0" />
+    <origin xyz="0.0 0.0 0.1725" rpy="0.0 0.0 0.0" />
   </joint>
 </robot>

Commit message: Added cervical links to urdf model

File: ur_description/urdf/ur5.urdf.xacro (robot description, xacro)
@@ -181,5 +181,5 @@
   <joint name="${prefix}base_joint" type="fixed">
     <axis xyz="0 0 1" />
-    <origin xyz="0.0 0.0 0.1725" rpy="0 0 -1.5708"/>
+    <origin xyz="0.0 0.0 0.1725" rpy="0 0 0"/>
     <parent link="${prefix}mobile_base"/>
     <child link="${prefix}base_link"/>
@@ -424,5 +424,5 @@
    <joint name="${prefix}gripper_joint" type="fixed">
     <axis xyz="0 1 0" />
-    <origin xyz="0.105 0.0 0.0" rpy="0 0 0"/>
+    <origin xyz="0.095 0.0 0.0" rpy="0 0 0"/>
     <parent link="${prefix}ee_link"/>
     <child link="${prefix}gripper"/>
@@ -432,14 +432,14 @@
       <origin xyz="0 0 0" rpy="0 0 0" />
       <geometry>
-          <box size="0.19 0.065 0.04"/>
-      </geometry>
-     <material name="black">
-        <color rgba="0.05 0.05 0.05 1"/>
-      </material>
-    </visual>
-	<collision>
-		<origin xyz="0 0 0" rpy="0 0 0" />
-		<geometry>
-          <box size="0.19 0.065 0.04"/>
+          <box size="0.225 0.065 0.04"/>
+      </geometry>
+     <material name="black">
+        <color rgba="0.05 0.05 0.05 1"/>
+      </material>
+    </visual>
+	<collision>
+		<origin xyz="0 0 0" rpy="0 0 0" />
+		<geometry>
+          <box size="0.225 0.065 0.04"/>
 		</geometry>
 	</collision>
@@ -513,4 +513,63 @@
     </sensor>
   </gazebo>
+   <!-- cervical links -->
+   <joint name="${prefix}cervical1_joint" type="fixed">
+    <axis xyz="0 1 0" />
+    <origin xyz="0.09 0.0 0.2" rpy="0 0 0"/>
+    <parent link="${prefix}upper_arm_link"/>
+    <child link="${prefix}cervical1_link"/>
+  </joint>
+  <link name="${prefix}cervical1_link">
+    <visual>
+      <origin xyz="0 0 0" rpy="0 0 0" />
+      <geometry>
+          <box size="0.08 0.06 0.23"/>
+      </geometry>
+     <material name="black">
+        <color rgba="0.05 0.05 0.05 1"/>
+      </material>
+    </visual>
+	<collision>
+		<origin xyz="0 0 0" rpy="0 0 0" />
+		<geometry>
+          <box size="0.08 0.06 0.23"/>
+		</geometry>
+	</collision>
+	<inertial>
+		<mass value="0.01" />
+		<inertia ixx="0.01" ixy="0.0" ixz="0.0"
+				iyy="0.01" iyz="0.0"
+				izz="0.01" />
+	</inertial>
+  </link>
+   <joint name="${prefix}cervical2_joint" type="fixed">
+    <axis xyz="0 1 0" />
+    <origin xyz="0.0 -0.08 0.205" rpy="0 0 0"/>
+    <parent link="${prefix}forearm_link"/>
+    <child link="${prefix}cervical2_link"/>
+  </joint>
+  <link name="${prefix}cervical2_link">
+    <visual>
+      <origin xyz="0 0 0" rpy="0 0 0" />
+      <geometry>
+          <box size="0.06 0.08 0.27"/>
+      </geometry>
+     <material name="black">
+        <color rgba="0.05 0.05 0.05 1"/>
+      </material>
+    </visual>
+	<collision>
+		<origin xyz="0 0 0" rpy="0 0 0" />
+		<geometry>
+          <box size="0.06 0.08 0.27"/>
+		</geometry>
+	</collision>
+	<inertial>
+		<mass value="0.01" />
+		<inertia ixx="0.01" ixy="0.0" ixz="0.0"
+				iyy="0.01" iyz="0.0"
+				izz="0.01" />
+	</inertial>
+  </link>
   </xacro:macro>
 </robot>

Commit message: Fixed gripper length

File: ur_description/urdf/ur5.urdf.xacro (robot description, xacro)
@@ -424,5 +424,5 @@
    <joint name="${prefix}gripper_joint" type="fixed">
     <axis xyz="0 1 0" />
-    <origin xyz="0.095 0.0 0.0" rpy="0 0 0"/>
+    <origin xyz="0.125 0.0 0.0" rpy="0 0 0"/>
     <parent link="${prefix}ee_link"/>
     <child link="${prefix}gripper"/>
@@ -432,14 +432,14 @@
       <origin xyz="0 0 0" rpy="0 0 0" />
       <geometry>
-          <box size="0.225 0.065 0.04"/>
-      </geometry>
-     <material name="black">
-        <color rgba="0.05 0.05 0.05 1"/>
-      </material>
-    </visual>
-	<collision>
-		<origin xyz="0 0 0" rpy="0 0 0" />
-		<geometry>
-          <box size="0.225 0.065 0.04"/>
+          <box size="0.25 0.065 0.04"/>
+      </geometry>
+     <material name="black">
+        <color rgba="0.05 0.05 0.05 1"/>
+      </material>
+    </visual>
+	<collision>
+		<origin xyz="0 0 0" rpy="0 0 0" />
+		<geometry>
+          <box size="0.25 0.065 0.04"/>
 		</geometry>
 	</collision>

Commit message: last modifies 16.04

File: ur_description/urdf/ur5.urdf.xacro (robot description, xacro)
@@ -92,4 +92,35 @@
 	</inertial>
   </link>
+<!--
+  <joint name="${prefix}gps_joint" type="fixed">
+    <axis xyz="0 0 1" />
+    <origin xyz="-0.1275 -0.2275 0.35" rpy="0 0 0"/>
+    <parent link="${prefix}mobile_base"/>
+    <child link="${prefix}gps_link"/>
+  </joint>
+   <link name="${prefix}gps_link">
+    <visual>
+      <origin xyz="0 0 0" rpy="0 0 0" />
+      <geometry>
+          <box size="0.15 0.15 0.3"/>
+      </geometry>
+     <material name="black">
+        <color rgba="0.05 0.05 0.05 1"/>
+      </material>
+    </visual>
+	<collision>
+		<origin xyz="0 0 0" rpy="0 0 0" />
+		<geometry>
+          <box size="0.15 0.15 0.3"/>
+		</geometry>
+	</collision>
+	<inertial>
+		<mass value="100" />
+		<inertia ixx="1" ixy="0.0" ixz="0.0"
+				iyy="1" iyz="0.0"
+				izz="1" />
+	</inertial>
+  </link>
+-->
   <joint name="${prefix}right_wheels_joint" type="fixed">
     <axis xyz="0 0 1" />
@@ -181,5 +212,5 @@
   <joint name="${prefix}base_joint" type="fixed">
     <axis xyz="0 0 1" />
-    <origin xyz="0.0 0.0 0.1725" rpy="0 0 0"/>
+    <origin xyz="0.0 0.0 0.1725" rpy="0 0 1.5708"/>
     <parent link="${prefix}mobile_base"/>
     <child link="${prefix}base_link"/>
@@ -451,16 +482,16 @@
 	</inertial>
   </link>
-  <joint name="${prefix}hokuyo_joint" type="fixed">
+  <joint name="${prefix}laser_joint" type="fixed">
     <axis xyz="0 1 0" />
-    <origin xyz="-0.05 0.0 0.03" rpy="0 0 0"/>
+    <origin xyz="-0.04 0.0 0.04" rpy="0 0 0"/>
     <parent link="${prefix}gripper"/>
-    <child link="${prefix}hokuyo_link"/>
-  </joint>
-  <!-- Hokuyo Laser -->
-  <link name="${prefix}hokuyo_link">
+    <child link="${prefix}laser_link"/>
+  </joint>
+  <!-- Laser -->
+  <link name="${prefix}laser_link">
     <collision>
       <origin xyz="0 0 0" rpy="0 0 0"/>
       <geometry>
-    <box size="0.1 0.1 0.1"/>
+    <box size="0.08 0.05 0.05"/>
       </geometry>
     </collision>
@@ -468,49 +499,62 @@
       <origin xyz="0 0 0" rpy="0 0 0"/>
       <geometry>
-        <mesh filename="package://ur_description/meshes/hokuyo.dae"/>
-      </geometry>
+        <box size="0.08 0.05 0.05"/>
+      </geometry>
+      <material name="black">
+        <color rgba="0.05 0.05 0.05 1"/>
+      </material>
     </visual>
     <inertial>
-      <mass value="1e-5" />
+		<mass value="0.01" />
+		<inertia ixx="0.01" ixy="0.0" ixz="0.0"
+				iyy="0.01" iyz="0.0"
+				izz="0.01" />
+	</inertial>
+  </link>
+  <joint name="${prefix}camera_joint" type="fixed">
+    <axis xyz="0 1 0" />
+    <origin xyz="-0.02 0.0 -0.04" rpy="0 0 0"/>
+    <parent link="${prefix}gripper"/>
+    <child link="${prefix}camera_link"/>
+  </joint>
+  <!-- Camera -->
+  <link name="${prefix}camera_link">
+    <collision>
       <origin xyz="0 0 0" rpy="0 0 0"/>
-      <inertia ixx="1e-6" ixy="0" ixz="0" iyy="1e-6" iyz="0" izz="1e-6" />
-    </inertial>
-  </link>
-  <!-- hokuyo -->
-  <gazebo reference="${prefix}hokuyo_link">
-    <sensor type="gpu_ray" name="head_hokuyo_sensor">
-      <pose>0 0 0 0 0 0</pose>
-      <visualize>false</visualize>
-      <update_rate>40</update_rate>
-      <ray>
-        <scan>
-          <horizontal>
-            <samples>720</samples>
-            <resolution>1</resolution>
-            <min_angle>-1.570796</min_angle>
-            <max_angle>1.570796</max_angle>
-          </horizontal>
-        </scan>
-        <range>
-          <min>0.10</min>
-          <max>10.0</max>
-          <resolution>0.01</resolution>
-        </range>
-        <noise>
-          <type>gaussian</type>
-          <!-- Noise parameters based on published spec for Hokuyo laser
-               achieving "+-30mm" accuracy at range < 10m.  A mean of 0.0m and
-               stddev of 0.01m will put 99.7% of samples within 0.03m of the true
-               reading. -->
-          <mean>0.0</mean>
-          <stddev>0.01</stddev>
-        </noise>
-      </ray>
-      <plugin name="gazebo_ros_head_hokuyo_controller" filename="libgazebo_ros_gpu_laser.so">
-        <topicName>/hokuyo/laser/scan</topicName>
-        <frameName>hokuyo_link</frameName>
-      </plugin>
-    </sensor>
-  </gazebo>
+      <geometry>
+    <box size="0.12 0.05 0.1"/>
+      </geometry>
+    </collision>
+    <visual>
+      <origin xyz="0 0 0" rpy="0 0 0"/>
+      <geometry>
+    <box size="0.12 0.05 0.1"/>
+      </geometry>
+      <material name="black">
+        <color rgba="0.05 0.05 0.05 1"/>
+      </material>
+    </visual>
+    <inertial>
+		<mass value="0.01" />
+		<inertia ixx="0.01" ixy="0.0" ixz="0.0"
+				iyy="0.01" iyz="0.0"
+				izz="0.01" />
+	</inertial>
+  </link>
+  <!-- sf30 -->
+  <joint name="${prefix}sf30_joint" type="fixed">
+    <axis xyz="0 1 0" />
+    <origin xyz="0.12 0.0 0.05" rpy="0 0 0"/>
+    <parent link="${prefix}ee_link"/>
+    <child link="sf30"/>
+  </joint>
+    <link name="sf30">
+      <collision>
+        <geometry>
+          <box size="0.01 0.01 0.01"/>
+        </geometry>
+        <origin rpy="0 0 0" xyz="-0.01 0 0"/>
+      </collision>
+    </link>
    <!-- cervical links -->
    <joint name="${prefix}cervical1_joint" type="fixed">
