Commit message: Downgrade to 14.04

File: ur_description/urdf/ur5.urdf.xacro (robot description, xacro)
@@ -482,4 +482,5 @@
 	</inertial>
   </link>
+<!--
   <joint name="${prefix}laser_joint" type="fixed">
     <axis xyz="0 1 0" />
@@ -488,5 +489,7 @@
     <child link="${prefix}laser_link"/>
   </joint>
+-->
   <!-- Laser -->
+<!--
   <link name="${prefix}laser_link">
     <collision>
@@ -512,7 +515,72 @@
 	</inertial>
   </link>
+-->
+  <joint name="${prefix}hokuyo_joint" type="fixed">
+     <axis xyz="0 1 0" />
+    <origin xyz="-0.05 0.0 0.06" rpy="0 0 0"/>
+     <parent link="${prefix}gripper"/>
+    <child link="${prefix}hokuyo_link"/>
+   </joint>
+  <!-- Hokuyo Laser -->
+  <link name="${prefix}hokuyo_link">
+     <collision>
+       <origin xyz="0 0 0" rpy="0 0 0"/>
+       <geometry>
+    <box size="0.08 0.05 0.05"/>
+       </geometry>
+     </collision>
+     <visual>
+       <origin xyz="0 0 0" rpy="0 0 0"/>
+       <geometry>
+        <mesh filename="package://ur_description/meshes/hokuyo.dae"/>
+       </geometry>
+      <material name="black">
+        <color rgba="0.05 0.05 0.05 1"/>
+      </material>
+     </visual>
+     <inertial>
+      <mass value="1e-5" />
+		<inertia ixx="1e-6" ixy="0" ixz="0" iyy="1e-6" iyz="0" izz="1e-6" />
+     </inertial>
+  </link>
+  <!-- hokuyo -->
+  <gazebo reference="${prefix}hokuyo_link">
+    <sensor type="ray" name="head_hokuyo_sensor">
+      <pose>0 0 0 0 0 0</pose>
+      <visualize>false</visualize>
+      <update_rate>40</update_rate>
+      <ray>
+        <scan>
+          <horizontal>
+            <samples>720</samples>
+            <resolution>1</resolution>
+            <min_angle>-1.570796</min_angle>
+            <max_angle>1.570796</max_angle>
+          </horizontal>
+        </scan>
+        <range>
+          <min>0.10</min>
+          <max>40.0</max>
+          <resolution>15.0</resolution>
+        </range>
+        <noise>
+          <type>gaussian</type>
+          <!-- Noise parameters based on published spec for Hokuyo laser
+               achieving "+-30mm" accuracy at range < 10m.  A mean of 0.0m and
+               stddev of 0.01m will put 99.7% of samples within 0.03m of the true
+               reading. -->
+          <mean>0.0</mean>
+          <stddev>0.01</stddev>
+        </noise>
+      </ray>
+      <plugin name="gazebo_ros_head_hokuyo_controller" filename="libgazebo_ros_laser.so">
+        <topicName>/scan</topicName>
+        <frameName>hokuyo_link</frameName>
+      </plugin>
+    </sensor>
+  </gazebo>
   <joint name="${prefix}camera_joint" type="fixed">
     <axis xyz="0 1 0" />
-    <origin xyz="-0.02 0.0 -0.04" rpy="0 0 0"/>
+    <origin xyz="-0.02 0.0 -0.06" rpy="0 0 0"/>
     <parent link="${prefix}gripper"/>
     <child link="${prefix}camera_link"/>
@@ -543,4 +611,5 @@
   </link>
   <!-- sf30 -->
+<!--
   <joint name="${prefix}sf30_joint" type="fixed">
     <axis xyz="0 1 0" />
@@ -557,4 +626,5 @@
       </collision>
     </link>
+-->
    <!-- cervical links -->
    <joint name="${prefix}cervical1_joint" type="fixed">

Commit message: Added controller link

File: ur_description/urdf/ur5.urdf.xacro (robot description, xacro)
@@ -152,4 +152,33 @@
 	</inertial>
   </link>
+  <joint name="${prefix}controladora_joint" type="fixed">
+    <axis xyz="0 0 1" />
+    <origin xyz="0.0 -0.425 0.3475" rpy="0 0 0"/>
+    <parent link="${prefix}mobile_base"/>
+    <child link="${prefix}controladora"/>
+  </joint>
+   <link name="${prefix}controladora">
+    <visual>
+      <origin xyz="0 0 0" rpy="0 0 0" />
+      <geometry>
+          <box size="0.47 0.25 0.35"/>
+      </geometry>
+     <material name="black">
+        <color rgba="0.05 0.05 0.05 1"/>
+      </material>
+    </visual>
+	<collision>
+		<origin xyz="0 0 0" rpy="0 0 0" />
+		<geometry>
+          <box size="0.18 0.605 0.4"/>
+		</geometry>
+	</collision>
+	<inertial>
+		<mass value="100" />
+		<inertia ixx="1" ixy="0.0" ixz="0.0"
+				iyy="1" iyz="0.0"
+				izz="1" />
+	</inertial>
+  </link>
   <joint name="${prefix}left_wheels_joint" type="fixed">
     <axis xyz="0 0 1" />
